Commit message: change robot cover, gazebo parameters

File: burger_war/models/blue_bot.urdf.xacro (robot description, xacro)
@@ -6,5 +6,5 @@
   <xacro:include filename="$(find burger_war)/models/burger_bot_common.xacro"/>
   <joint name="tag1_joint" type="fixed">
-    <origin rpy="-1.571 3.1415 0" xyz="-0.03 0.07 0.09"/>
+    <origin rpy="-1.571 3.1415 0" xyz="-0.032 0.09 0.1"/>
     <parent link="base_link"/>
     <child link="tag1"/>
@@ -19,5 +19,5 @@
   </link>
   <joint name="tag1-1_joint" type="fixed">
-    <origin rpy="-1.571 3.1415 0" xyz="-0.03 0.069 0.09"/>
+    <origin rpy="-1.571 3.1415 0" xyz="-0.032 0.089 0.1"/>
     <parent link="base_link"/>
     <child link="tag1-1"/>
@@ -31,5 +31,5 @@
   </link>
   <joint name="tag2_joint" type="fixed">
-    <origin rpy="1.571 0 0" xyz="-0.03 -0.07 0.09"/>
+    <origin rpy="1.571 0 0" xyz="-0.032 -0.09 0.1"/>
     <parent link="base_link"/>
     <child link="tag2"/>
@@ -43,5 +43,5 @@
   </link>
   <joint name="tag2-1_joint" type="fixed">
-    <origin rpy="1.571 0 0" xyz="-0.03 -0.069 0.09"/>
+    <origin rpy="1.571 0 0" xyz="-0.032 -0.089 0.1"/>
     <parent link="base_link"/>
     <child link="tag2-1"/>
@@ -55,5 +55,5 @@
   </link>
   <joint name="tag3_joint" type="fixed">
-    <origin rpy="1.571 0 -1.571" xyz="-0.101 0.0 0.09"/>
+    <origin rpy="1.571 0 -1.571" xyz="-0.122 0.0 0.1"/>
     <parent link="base_link"/>
     <child link="tag3"/>
@@ -67,5 +67,5 @@
   </link>
   <joint name="tag3-1_joint" type="fixed">
-    <origin rpy="1.571 0 -1.571" xyz="-0.10 0.0 0.09"/>
+    <origin rpy="1.571 0 -1.571" xyz="-0.121 0.0 0.1"/>
     <parent link="base_link"/>
     <child link="tag3-1"/>

File: burger_war/models/burger_bot_common.xacro (robot description, xacro)
@@ -9,22 +9,30 @@
   <link name="base_link">
     <visual>
-      <origin xyz="-0.032 0 0.0" rpy="0 0 0"/>
-      <geometry>
-        <mesh filename="package://turtlebot3_description/meshes/bases/burger_base.stl" scale="0.001 0.001 0.001"/>
+      <!--<origin xyz="-0.032 0 0.0" rpy="0 0 0"/>-->
+      <origin xyz="-0.032 0 0.00875" rpy="0 0 0"/>
+      <geometry>
+        <!--<mesh filename="package://turtlebot3_description/meshes/bases/burger_base.stl" scale="0.001 0.001 0.001"/>-->
+        <mesh filename="model://burger_bot/burger_bot_cover.stl" scale="0.001 0.001 0.001"/>
       </geometry>
       <material name="light_black"/>
     </visual>
     <collision>
-      <origin xyz="-0.032 0 0.070" rpy="0 0 0"/>
-      <geometry>
-        <box size="0.140 0.140 0.12"/> <!-- <box size="0.140 0.140 0.143"/> -->
-      </geometry>
-    </collision>
-    <inertial>
-      <origin xyz="0 0 0" rpy="0 0 0"/>
-      <mass value="8.2573504e-01"/>
+      <origin xyz="-0.032 0 0.07875" rpy="0 0 0"/>
+      <geometry>
+        <box size="0.178 0.116 0.13"/> <!-- <box size="0.140 0.140 0.143"/> -->
+      </geometry>
+    </collision>
+    <inertial>
+      <!--<origin xyz="0 0 0" rpy="0 0 0"/>-->
+      <origin xyz="-0.032 0 0.07" rpy="0 0 0"/>
+      <mass value="2.6"/><!--<mass value="8.2573504e-01"/>-->
+      <!--
       <inertia ixx="2.2124416e-03" ixy="-1.2294101e-05" ixz="3.4938785e-05"
                iyy="2.1193702e-03" iyz="-5.0120904e-06"
                izz="2.0064271e-03" />
+               -->
+      <inertia ixx="6.65340e-03" ixy="0" ixz="0"
+               iyy="6.65340e-03" iyz="0"
+               izz="8.25240e-03" />
     </inertial>
   </link>
@@ -97,5 +105,6 @@
     </visual>
     <collision>
-      <origin xyz="0 0.00625 0" rpy="0 0 0"/>
+      <!--<origin xyz="0 0.00625 0" rpy="0 0 0"/>-->
+      <origin xyz="0 0 0" rpy="0 0 0"/>
       <geometry>
         <!--<box size="0.030 0.009 0.020"/>-->
@@ -105,5 +114,5 @@
     <inertial>
       <origin xyz="0 0 0" />
-      <mass value="0.5" /> <!--<mass value="0.005" />-->
+      <mass value="0.05" /> <!--<mass value="0.5" /><mass value="0.005" />-->
       <inertia ixx="0.001" ixy="0.0" ixz="0.0"
                iyy="0.001" iyz="0.0"
@@ -120,5 +129,6 @@
     <parent link="base_link"/>
     <child link="base_scan"/>
-    <origin xyz="-0.032 0 0.172" rpy="0 0 0"/>
+    <!--<origin xyz="-0.032 0 0.172" rpy="0 0 0"/>-->
+    <origin xyz="-0.032 0 0.16855" rpy="0 0 0"/>
   </joint>
   <link name="base_scan">
@@ -147,15 +157,19 @@
     <parent link="base_link"/>
     <child link="base_camera"/>
-    <origin xyz="0.03 0 0.1" rpy="-1.57 0 -1.57"/>
+    <!--<origin xyz="0.03 0 0.1" rpy="-1.57 0 -1.57"/>-->
+    <origin xyz="0.055 0 0.1" rpy="-1.57 0 -1.57"/>
   </joint>
   <link name="base_camera">
     <visual>
-      <origin xyz="0 0 0.0" rpy="0 0 0"/>
+      <origin xyz="0 0 -0.01" rpy="0 0 0"/>
       <geometry>
         <box size="0.03 0.01 0.01"/>
       </geometry>
-      <material name="dark"/>
-    </visual>
-  </link>
+      <!--<material name="dark"/>-->
+    </visual>
+  </link>
+  <gazebo reference="base_camera">
+    <material>Gazebo/Grey</material>
+  </gazebo>
   <joint name="poll_joint" type="fixed">
     <origin rpy="0 0 0" xyz="-0.09 0.0 0.21"/>

File: burger_war/models/red_bot.urdf.xacro (robot description, xacro)
@@ -6,5 +6,6 @@
   <xacro:include filename="$(find burger_war)/models/burger_bot_common.xacro"/>
   <joint name="tag1_joint" type="fixed">
-    <origin rpy="-1.571 3.1415 0" xyz="-0.03 0.07 0.09"/>
+    <!--<origin rpy="-1.571 3.1415 0" xyz="-0.03 0.07 0.09"/>-->
+    <origin rpy="-1.571 3.1415 0" xyz="-0.032 0.09 0.1"/>
     <parent link="base_link"/>
     <child link="tag1"/>
@@ -19,5 +20,6 @@
   </link>
   <joint name="tag1-1_joint" type="fixed">
-    <origin rpy="-1.571 3.1415 0" xyz="-0.03 0.069 0.09"/>
+    <!--<origin rpy="-1.571 3.1415 0" xyz="-0.03 0.069 0.09"/>-->
+    <origin rpy="-1.571 3.1415 0" xyz="-0.032 0.089 0.1"/>
     <parent link="base_link"/>
     <child link="tag1-1"/>
@@ -31,5 +33,6 @@
   </link>
   <joint name="tag2_joint" type="fixed">
-    <origin rpy="1.571 0 0" xyz="-0.03 -0.07 0.09"/>
+    <!--<origin rpy="1.571 0 0" xyz="-0.03 -0.07 0.09"/>-->
+    <origin rpy="1.571 0 0" xyz="-0.032 -0.09 0.1"/>
     <parent link="base_link"/>
     <child link="tag2"/>
@@ -43,5 +46,6 @@
   </link>
   <joint name="tag2-1_joint" type="fixed">
-    <origin rpy="1.571 0 0" xyz="-0.03 -0.069 0.09"/>
+    <!--<origin rpy="1.571 0 0" xyz="-0.03 -0.069 0.09"/>-->
+    <origin rpy="1.571 0 0" xyz="-0.032 -0.089 0.1"/>
     <parent link="base_link"/>
     <child link="tag2-1"/>
@@ -55,5 +59,6 @@
   </link>
   <joint name="tag3_joint" type="fixed">
-    <origin rpy="1.571 0 -1.571" xyz="-0.101 0.0 0.09"/>
+    <!--<origin rpy="1.571 0 -1.571" xyz="-0.101 0.0 0.09"/>-->
+    <origin rpy="1.571 0 -1.571" xyz="-0.122 0.0 0.1"/>
     <parent link="base_link"/>
     <child link="tag3"/>
@@ -67,5 +72,6 @@
   </link>
   <joint name="tag3-1_joint" type="fixed">
-    <origin rpy="1.571 0 -1.571" xyz="-0.10 0.0 0.09"/>
+    <!--<origin rpy="1.571 0 -1.571" xyz="-0.10 0.0 0.09"/>-->
+    <origin rpy="1.571 0 -1.571" xyz="-0.121 0.0 0.1"/>
     <parent link="base_link"/>
     <child link="tag3-1"/>
