Commit message: add Yellow disc

File: burger_war/models/burger_bot_common.xacro (robot description, xacro)
@@ -18,5 +18,5 @@
       <origin xyz="-0.032 0 0.070" rpy="0 0 0"/>
       <geometry>
-        <box size="0.140 0.140 0.143"/>
+        <box size="0.140 0.140 0.12"/> <!-- <box size="0.140 0.140 0.143"/> -->
       </geometry>
     </collision>
@@ -88,16 +88,22 @@
     <parent link="base_link"/>
     <child link="caster_back_link"/>
-    <origin xyz="-0.081 0 -0.004" rpy="-1.57 0 0"/>
+    <origin xyz="-0.074 0 0.0025" rpy="0 0 0"/><!--<origin xyz="-0.081 0 -0.004" rpy="-1.57 0 0"/>-->
   </joint>
   <link name="caster_back_link">
+    <visual>
+      <geometry>
+        <sphere radius="0.0125"/>
+      </geometry>
+    </visual>
     <collision>
-  <origin xyz="0 0.001 0" rpy="0 0 0"/>
+      <origin xyz="0 0.00625 0" rpy="0 0 0"/>
       <geometry>
-        <box size="0.030 0.009 0.020"/>
+        <!--<box size="0.030 0.009 0.020"/>-->
+        <sphere radius="0.0125"/>
       </geometry>
     </collision>
     <inertial>
       <origin xyz="0 0 0" />
-      <mass value="0.005" />
+      <mass value="0.5" /> <!--<mass value="0.005" />-->
       <inertia ixx="0.001" ixy="0.0" ixz="0.0"
                iyy="0.001" iyz="0.0"

File: burger_war/models/burgerbot.gazebo.xacro (robot description, xacro)
@@ -7,28 +7,30 @@
   </gazebo>
   <gazebo reference="wheel_left_link">
-    <mu1>0.1</mu1>
-    <mu2>0.1</mu2>
-    <kp>500000.0</kp>
-    <kd>10.0</kd>
+    <mu1>1</mu1>
+    <mu2>1</mu2>
+    <kp>10000000.0</kp>
+    <kd>100000.0</kd>
     <minDepth>0.001</minDepth>
-    <maxVel>0.1</maxVel>
-    <fdir1>1 0 0</fdir1>
+    <maxVel>0.0</maxVel>
+    <fdir1>0 0 0</fdir1>
     <material>Gazebo/FlatBlack</material>
   </gazebo>
   <gazebo reference="wheel_right_link">
-    <mu1>0.1</mu1> <mu2>0.1</mu2> <kp>500000.0</kp>
-    <kd>10.0</kd>
+    <mu1>1</mu1>
+    <mu2>1</mu2>
+    <kp>10000000.0</kp>
+    <kd>100000.0</kd>
     <minDepth>0.001</minDepth>
-    <maxVel>0.1</maxVel>
-    <fdir1>1 0 0</fdir1>
+    <maxVel>0.0</maxVel>
+    <fdir1>0 0 0</fdir1>
     <material>Gazebo/FlatBlack</material>
   </gazebo>
   <gazebo reference="caster_back_link">
-    <mu1>0.1</mu1>
-    <mu2>0.1</mu2>
-    <kp>1000000.0</kp>
-    <kd>100.0</kd>
+    <mu1>0.01</mu1>
+    <mu2>0.01</mu2>
+    <kp>10000000.0</kp>
+    <kd>100000.0</kd>
     <minDepth>0.001</minDepth>
-    <maxVel>1.0</maxVel>
+    <maxVel>0.0</maxVel>
     <material>Gazebo/FlatBlack</material>
   </gazebo>

Commit message: fix physical parameters

File: burger_war/models/burger_bot_common.xacro (robot description, xacro)
@@ -13,5 +13,5 @@
       <geometry>
         <!--<mesh filename="package://turtlebot3_description/meshes/bases/burger_base.stl" scale="0.001 0.001 0.001"/>-->
-        <mesh filename="model://burger_bot/burger_bot_cover.stl" scale="0.001 0.001 0.001"/>
+        <mesh filename="package://burger_war/models/burger_bot/burger_bot_cover.stl" scale="0.001 0.001 0.001"/>
       </geometry>
       <material name="light_black"/>
@@ -21,4 +21,40 @@
       <geometry>
         <box size="0.178 0.116 0.13"/> <!-- <box size="0.140 0.140 0.143"/> -->
+      </geometry>
+    </collision>
+    <collision>
+      <origin xyz="-0.032 0.0885 0.10125" rpy="0 0 0"/>
+      <geometry>
+        <box size="0.116 0.001 0.085"/>
+      </geometry>
+    </collision>
+    <collision>
+      <origin xyz="-0.032 -0.0885 0.10125" rpy="0 0 0"/>
+      <geometry>
+        <box size="0.116 0.001 0.085"/>
+      </geometry>
+    </collision>
+    <collision>
+      <origin xyz="-0.10535 0.07335 0.07875" rpy="0 0 0.785398163"/>
+      <geometry>
+        <box size="0.04243 0.001 0.13"/>
+      </geometry>
+    </collision>
+    <collision>
+      <origin xyz="-0.10535 -0.07335 0.07875" rpy="0 0 -0.785398163"/>
+      <geometry>
+        <box size="0.04243 0.001 0.13"/>
+      </geometry>
+    </collision>
+    <collision>
+      <origin xyz="0.04138 0.07335 0.10125" rpy="0 0 -0.785398163"/>
+      <geometry>
+        <box size="0.04243 0.001 0.085"/>
+      </geometry>
+    </collision>
+    <collision>
+      <origin xyz="0.04138 -0.07335 0.10125" rpy="0 0 0.785398163"/>
+      <geometry>
+        <box size="0.04243 0.001 0.085"/>
       </geometry>
     </collision>

File: burger_war/models/burgerbot.gazebo.xacro (robot description, xacro)
@@ -4,4 +4,10 @@
   <xacro:arg name="imu_visual"   default="false"/>
   <gazebo reference="base_link">
+    <mu1>0.01</mu1>
+    <mu2>0.01</mu2>
+    <kp>1000000.0</kp>
+    <kd>100.0</kd>
+    <minDepth>0.001</minDepth>
+    <maxVel>1.0</maxVel>
     <material>Gazebo/DarkGrey</material>
   </gazebo>
@@ -9,9 +15,9 @@
     <mu1>1</mu1>
     <mu2>1</mu2>
-    <kp>10000000.0</kp>
-    <kd>100000.0</kd>
+    <kp>500000.0</kp>
+    <kd>10.0</kd>
     <minDepth>0.001</minDepth>
-    <maxVel>0.0</maxVel>
-    <fdir1>0 0 0</fdir1>
+    <maxVel>0.1</maxVel>
+    <fdir1>1 0 0</fdir1>
     <material>Gazebo/FlatBlack</material>
   </gazebo>
@@ -19,9 +25,9 @@
     <mu1>1</mu1>
     <mu2>1</mu2>
-    <kp>10000000.0</kp>
-    <kd>100000.0</kd>
+    <kp>500000.0</kp>
+    <kd>10.0</kd>
     <minDepth>0.001</minDepth>
-    <maxVel>0.0</maxVel>
-    <fdir1>0 0 0</fdir1>
+    <maxVel>0.1</maxVel>
+    <fdir1>1 0 0</fdir1>
     <material>Gazebo/FlatBlack</material>
   </gazebo>
@@ -29,8 +35,8 @@
     <mu1>0.01</mu1>
     <mu2>0.01</mu2>
-    <kp>10000000.0</kp>
-    <kd>100000.0</kd>
+    <kp>1000000.0</kp>
+    <kd>100.0</kd>
     <minDepth>0.001</minDepth>
-    <maxVel>0.0</maxVel>
+    <maxVel>1.0</maxVel>
     <material>Gazebo/FlatBlack</material>
   </gazebo>
